File: fuel_gauge.kicad_sch (KiCad schematic)
At the start: 2 parts, among them U3 MAX17055EWL+T

Commit message: footprints
Parts:
- C_FG1: footprint (none) -> Capacitor_SMD:C_0402_1005Metric
- U3: footprint 21-100129A_W91N1+1_MXM -> MAX17055EWL+T:BGA9N40P3X3_140X149X69N
Changed lines of the file:
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@@
 			)
 		)
-		(property "Footprint" ""
+		(property "Footprint" "Capacitor_SMD:C_0402_1005Metric"
 			(at 107.6452 114.3 0)
 			(effects
@@
 			)
 		)
-		(property "Footprint" "21-100129A_W91N1+1_MXM"
+		(property "Footprint" "MAX17055EWL+T:BGA9N40P3X3_140X149X69N"
 			(at 114.3 88.9 0)
 			(effects
