File: UI.kicad_sch (KiCad schematic)
At the start: 4 parts, among them J4 Conn_01x12, J5 Conn_01x04

Commit message: footprints
Parts:
- C_DISP1: renamed from C_DISP; footprint (none) -> Capacitor_SMD:C_0402_1005Metric
- J4: footprint (none) -> Connector_JST:JST_GH_SM12B-GHS-TB_1x12-1MP_P1.25mm_Horizontal
- J5: footprint (none) -> Connector_JST:JST_XH_B4B-XH-A_1x04_P2.50mm_Vertical
- R22: footprint (none) -> Resistor_SMD:R_0402_1005Metric
Changed lines of the file:
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@@
 			)
 		)
-		(property "Footprint" ""
+		(property "Footprint" "Resistor_SMD:R_0402_1005Metric"
 			(at 99.822 69.85 90)
 			(effects
@@
 			)
 		)
-		(property "Footprint" ""
+		(property "Footprint" "Connector_JST:JST_GH_SM12B-GHS-TB_1x12-1MP_P1.25mm_Horizontal"
 			(at 132.08 39.37 0)
 			(effects
@@
 		(dnp no)
 		(fields_autoplaced yes)
-		(property "Reference" "C_DISP"
+		(property "Reference" "C_DISP1"
 			(at 109.22 29.2099 0)
 			(effects
@@
 			)
 		)
-		(property "Footprint" ""
+		(property "Footprint" "Capacitor_SMD:C_0402_1005Metric"
 			(at 106.3752 34.29 0)
 			(effects
@@
 			(project ""
 				(path "/96bcf3cc-a3b8-4386-8709-07acaf7b6253/ca908c34-ad55-48a6-bd0d-9c55747ba4f1"
-					(reference "C_DISP")
+					(reference "C_DISP1")
 					(unit 1)
 				)
@@
 			)
 		)
-		(property "Footprint" ""
+		(property "Footprint" "Connector_JST:JST_XH_B4B-XH-A_1x04_P2.50mm_Vertical"
 			(at 133.35 68.58 0)
 			(effects

Commit message: net labels
Connections:
- net FIRE_LED: now reaches J5.4 (Pin_4), R22.2
Changed lines of the file:
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@@
+		)
+	)
+	(label "FIRE_LED"
+		(at 114.2376 73.66 0)
+		(effects
+			(font
+				(size 1.27 1.27)
+			)
+			(justify left bottom)
 		)
 	)
