File: boost_converter.kicad_sch (KiCad schematic)
At the start: 15 parts, among them U4 TPS61088RHLR, U5 MCP4561-104E/MS

Commit message: finished schematics
Parts:
- added C_VSENSE: 100nF, symbol Device:C
- added R_DIV1: 100k, symbol Device:R
- added R_DIV2: 47k, symbol Device:R
Connections:
- net GND: now also C_VSENSE.2, R_DIV2.2
- net V_BOOST: now also R_DIV1.2
- new net V_SENSE: C_VSENSE.1, R_DIV1.1, R_DIV2.1

Commit message: footprints
Parts:
- C16: footprint (none) -> Capacitor_SMD:C_1206_3216Metric
- C17: footprint (none) -> Capacitor_SMD:C_0402_1005Metric
- C_BIN1, C_BOUT1, C_BOUT2: footprint (none) -> Capacitor_SMD:C_0805_2012Metric
- C_BOOT1: renamed from C_BOOT; footprint (none) -> Capacitor_SMD:C_0402_1005Metric
- C_COMP1: renamed from C_COMP; footprint (none) -> Capacitor_SMD:C_0402_1005Metric
- C_VCC1: renamed from C_VCC; footprint (none) -> Capacitor_SMD:C_0402_1005Metric
- C_VSENSE1: renamed from C_VSENSE; footprint (none) -> Capacitor_SMD:C_0402_1005Metric
- R4, R_DIV1, R_DIV2: footprint (none) -> Resistor_SMD:R_0402_1005Metric
- R_COMP1: renamed from R_COMP; footprint (none) -> Resistor_SMD:R_0402_1005Metric
- R_ILIM1: renamed from R_ILIM; footprint (none) -> Resistor_SMD:R_0402_1005Metric
- R_SAFE1: renamed from R_SAFE; footprint (none) -> Resistor_SMD:R_0402_1005Metric
- U11: renamed from U5; footprint MSOP8_MC_MCH -> Package_SO:SOIC-8_3.9x4.9mm_P1.27mm
- U4: footprint RHL0020A -> Package_DFN_QFN:QFN-20-1EP_4x4mm_P0.5mm_EP2.7x2.7mm_ThermalVias
Changed lines of the file:
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@@
 			)
 		)
-		(property "Footprint" ""
+		(property "Footprint" "Capacitor_SMD:C_0805_2012Metric"
 			(at 107.6452 113.03 0)
 			(effects
@@
 		(dnp no)
 		(fields_autoplaced yes)
-		(property "Reference" "R_COMP"
+		(property "Reference" "R_COMP1"
 			(at 30.48 99.0599 0)
 			(effects
@@
 			)
 		)
-		(property "Footprint" ""
+		(property "Footprint" "Resistor_SMD:R_0402_1005Metric"
 			(at 26.162 100.33 90)
 			(effects
@@
 			(project ""
 				(path "/96bcf3cc-a3b8-4386-8709-07acaf7b6253/e1164715-2b15-4b84-b46a-089d56ad88f2"
-					(reference "R_COMP")
+					(reference "R_COMP1")
 					(unit 1)
 				)
@@
 		(dnp no)
 		(fields_autoplaced yes)
-		(property "Reference" "R_SAFE"
+		(property "Reference" "R_SAFE1"
 			(at 85.09 119.3799 0)
 			(effects
@@
 			)
 		)
-		(property "Footprint" ""
+		(property "Footprint" "Resistor_SMD:R_0402_1005Metric"
 			(at 80.772 120.65 90)
 			(effects
@@
 			(project ""
 				(path "/96bcf3cc-a3b8-4386-8709-07acaf7b6253/e1164715-2b15-4b84-b46a-089d56ad88f2"
-					(reference "R_SAFE")
+					(reference "R_SAFE1")
 					(unit 1)
 				)
@@
 			)
 		)
-		(property "Footprint" ""
+		(property "Footprint" "Capacitor_SMD:C_1206_3216Metric"
 			(at 147.0152 113.03 0)
 			(effects
@@
 		(dnp no)
 		(fields_autoplaced yes)
-		(property "Reference" "C_VSENSE"
+		(property "Reference" "C_VSENSE1"
 			(at 161.29 90.1699 0)
 			(effects
@@
 			)
 		)
-		(property "Footprint" ""
+		(property "Footprint" "Capacitor_SMD:C_0402_1005Metric"
 			(at 158.4452 95.25 0)
 			(effects
@@
 			(project ""
 				(path "/96bcf3cc-a3b8-4386-8709-07acaf7b6253/e1164715-2b15-4b84-b46a-089d56ad88f2"
-					(reference "C_VSENSE")
+					(reference "C_VSENSE1")
 					(unit 1)
 				)
@@
 		(dnp no)
 		(fields_autoplaced yes)
-		(property "Reference" "C_COMP"
+		(property "Reference" "C_COMP1"
 			(at 25.4 99.0599 0)
 			(effects
@@
 			)
 		)
-		(property "Footprint" ""
+		(property "Footprint" "Capacitor_SMD:C_0402_1005Metric"
 			(at 22.5552 104.14 0)
 			(effects
@@
 			(project ""
 				(path "/96bcf3cc-a3b8-4386-8709-07acaf7b6253/e1164715-2b15-4b84-b46a-089d56ad88f2"
-					(reference "C_COMP")
+					(reference "C_COMP1")
 					(unit 1)
 				)
@@
 		(dnp no)
 		(fields_autoplaced yes)
-		(property "Reference" "U5"
+		(property "Reference" "U11"
 			(at 146.05 59.69 0)
 			(effects
@@
 			)
 		)
-		(property "Footprint" "MSOP8_MC_MCH"
+		(property "Footprint" "Package_SO:SOIC-8_3.9x4.9mm_P1.27mm"
 			(at 115.57 69.85 0)
 			(effects
@@
 			(project ""
 				(path "/96bcf3cc-a3b8-4386-8709-07acaf7b6253/e1164715-2b15-4b84-b46a-089d56ad88f2"
-					(reference "U5")
+					(reference "U11")
 					(unit 1)
 				)
@@
 			)
 		)
-		(property "Footprint" "RHL0020A"
+		(property "Footprint" "Package_DFN_QFN:QFN-20-1EP_4x4mm_P0.5mm_EP2.7x2.7mm_ThermalVias"
 			(at 52.07 102.87 0)
 			(effects
@@
 		(dnp no)
 		(fields_autoplaced yes)
-		(property "Reference" "R_ILIM"
+		(property "Reference" "R_ILIM1"
 			(at 31.75 106.6799 0)
 			(effects
@@
 			)
 		)
-		(property "Footprint" ""
+		(property "Footprint" "Resistor_SMD:R_0402_1005Metric"
 			(at 27.432 107.95 90)
 			(effects
@@
 			(project ""
 				(path "/96bcf3cc-a3b8-4386-8709-07acaf7b6253/e1164715-2b15-4b84-b46a-089d56ad88f2"
-					(reference "R_ILIM")
+					(reference "R_ILIM1")
 					(unit 1)
 				)
@@
 			)
 		)
-		(property "Footprint" ""
+		(property "Footprint" "Capacitor_SMD:C_0805_2012Metric"
 			(at 126.6952 113.03 0)
 			(effects
@@
 		(dnp no)
 		(fields_autoplaced yes)
-		(property "Reference" "C_VCC"
+		(property "Reference" "C_VCC1"
 			(at 30.48 82.5499 0)
 			(effects
@@
 			)
 		)
-		(property "Footprint" ""
+		(property "Footprint" "Capacitor_SMD:C_0402_1005Metric"
 			(at 27.6352 87.63 0)
 			(effects
@@
 			(project ""
 				(path "/96bcf3cc-a3b8-4386-8709-07acaf7b6253/e1164715-2b15-4b84-b46a-089d56ad88f2"
-					(reference "C_VCC")
+					(reference "C_VCC1")
 					(unit 1)
 				)
@@
 			)
 		)
-		(property "Footprint" ""
+		(property "Footprint" "Capacitor_SMD:C_0402_1005Metric"
 			(at 25.0952 116.84 0)
 			(effects
@@
 			)
 		)
-		(property "Footprint" ""
+		(property "Footprint" "Resistor_SMD:R_0402_1005Metric"
 			(at 68.072 113.03 90)
 			(effects
@@
 			)
 		)
-		(property "Footprint" ""
+		(property "Footprint" "Capacitor_SMD:C_0805_2012Metric"
 			(at 25.0952 76.2 0)
 			(effects
@@
 			)
 		)
-		(property "Footprint" ""
+		(property "Footprint" "Resistor_SMD:R_0402_1005Metric"
 			(at 170.942 91.44 90)
 			(effects
@@
 		(dnp no)
 		(fields_autoplaced yes)
-		(property "Reference" "C_BOOT"
+		(property "Reference" "C_BOOT1"
 			(at 80.01 80.0099 0)
 			(effects
@@
 			)
 		)
-		(property "Footprint" ""
+		(property "Footprint" "Capacitor_SMD:C_0402_1005Metric"
 			(at 77.1652 85.09 0)
 			(effects
@@
 			(project ""
 				(path "/96bcf3cc-a3b8-4386-8709-07acaf7b6253/e1164715-2b15-4b84-b46a-089d56ad88f2"
-					(reference "C_BOOT")
+					(reference "C_BOOT1")
 					(unit 1)
 				)
@@
 			)
 		)
-		(property "Footprint" ""
+		(property "Footprint" "Resistor_SMD:R_0402_1005Metric"
 			(at 145.542 91.44 90)
 			(effects

Commit message: net labels
Connections:
- net BOOST_COMP: now reaches R_COMP1.1, U4.18 (COMP)
- net BOOST_COMP: now also C_COMP1.2, R_COMP1.2
- net DPOT_WIPER: now reaches R4.2, R_SAFE1.1, U11.6 (P0W), U4.17 (FB)
- net BOOST_SW: now reaches C_BOOT1.2, L2.1, U4.4 (SW), U4.5 (SW), U4.6 (SW), U4.7 (SW)
- net BOOST_VCC: now reaches C_VCC1.1, U4.1 (VCC)
- net BOOST_SS: now reaches C17.1, U4.10 (SS)
- net BOOST_ILIM: now reaches R_ILIM1.1, U4.19 (ILIM)
- net BOOST_BOOT: now reaches C_BOOT1.1, U4.8 (BOOT)
Changed lines of the file:
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@@
+		)
+	)
+	(label "DPOT_WIPER"
+		(at 176.53 86.505 0)
+		(effects
+			(font
+				(size 1.27 1.27)
+			)
+			(justify left bottom)
+		)
+	)
+	(label "BOOST_SS"
+		(at 32.1859 113.03 0)
+		(effects
+			(font
+				(size 1.27 1.27)
+			)
+			(justify left bottom)
+		)
+	)
+	(label "BOOST_BOOT"
+		(at 71.9385 77.47 0)
+		(effects
+			(font
+				(size 1.27 1.27)
+			)
+			(justify left bottom)
+		)
+	)
+	(label "BOOST_COMP"
+		(at 23.8381 104.14 0)
+		(effects
+			(font
+				(size 1.27 1.27)
+			)
+			(justify left bottom)
+		)
+	)
+	(label "BOOST_SW"
+		(at 76.2 87.63 0)
+		(effects
+			(font
+				(size 1.27 1.27)
+			)
+			(justify left bottom)
+		)
+	)
+	(label "BOOST_ILIM"
+		(at 31.6034 107.95 0)
+		(effects
+			(font
+				(size 1.27 1.27)
+			)
+			(justify left bottom)
+		)
+	)
+	(label "BOOST_VCC"
+		(at 29.8806 82.55 0)
+		(effects
+			(font
+				(size 1.27 1.27)
+			)
+			(justify left bottom)
+		)
+	)
+	(label "BOOST_COMP"
+		(at 31.4854 100.33 0)
+		(effects
+			(font
+				(size 1.27 1.27)
+			)
+			(justify left bottom)
 		)
 	)
