File: safety_logic.kicad_sch (KiCad schematic)
At the start: 16 parts, among them U12 74LVC1G17, U13 74LVC1G04, U6 NE555DR, U7 74LVC08APW

Commit message: footprints
Parts:
- C15: footprint (none) -> Capacitor_SMD:C_0805_2012Metric
- C_555: footprint (none) -> Capacitor_SMD:C_0402_1005Metric
- C_AND1: renamed from C_AND; footprint (none) -> Capacitor_SMD:C_0402_1005Metric
- C_CV1: renamed from C_CV; footprint (none) -> Capacitor_SMD:C_0402_1005Metric
- C_DEBOUNCE1: renamed from C_DEBOUNCE; footprint (none) -> Capacitor_SMD:C_0402_1005Metric
- C_INV1: renamed from C_INV; footprint (none) -> Capacitor_SMD:C_0402_1005Metric
- C_SCHMITT1: renamed from C_SCHMITT; footprint (none) -> Capacitor_SMD:C_0402_1005Metric
- R11, R12: footprint (none) -> Resistor_SMD:R_0402_1005Metric
- R3: footprint (none) -> Resistor_SMD:R_0603_1608Metric
- R_ALERT1: renamed from R_ALERT; footprint (none) -> Resistor_SMD:R_0402_1005Metric
- R_DEBOUNCE1: renamed from R_DEBOUNCE; footprint (none) -> Resistor_SMD:R_0402_1005Metric
- U12, U13: footprint (none) -> Package_TO_SOT_SMD:SOT-353_SC-70-5
- U6: footprint D8 -> Package_SO:SOIC-8_3.9x4.9mm_P1.27mm
- U7: footprint SOT402-1_NXP -> Package_SO:TSSOP-14_4.4x5mm_P0.65mm
Changed lines of the file:
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@@
 			)
 		)
-		(property "Footprint" "D8"
+		(property "Footprint" "Package_SO:SOIC-8_3.9x4.9mm_P1.27mm"
 			(at 43.18 50.8 0)
 			(effects
@@
 			)
 		)
-		(property "Footprint" ""
+		(property "Footprint" "Capacitor_SMD:C_0805_2012Metric"
 			(at 119.0752 64.77 0)
 			(effects
@@
 		(dnp no)
 		(fields_autoplaced yes)
-		(property "Reference" "C_CV"
+		(property "Reference" "C_CV1"
 			(at 113.03 63.4999 0)
 			(effects
@@
 			)
 		)
-		(property "Footprint" ""
+		(property "Footprint" "Capacitor_SMD:C_0402_1005Metric"
 			(at 110.1852 68.58 0)
 			(effects
@@
 			(project ""
 				(path "/96bcf3cc-a3b8-4386-8709-07acaf7b6253/b707efaf-e934-4479-b5a7-a53392b0d81d"
-					(reference "C_CV")
+					(reference "C_CV1")
 					(unit 1)
 				)
@@
 		(dnp no)
 		(fields_autoplaced yes)
-		(property "Reference" "C_INV"
+		(property "Reference" "C_INV1"
 			(at 186.69 120.6499 0)
 			(effects
@@
 			)
 		)
-		(property "Footprint" ""
+		(property "Footprint" "Capacitor_SMD:C_0402_1005Metric"
 			(at 183.8452 125.73 0)
 			(effects
@@
 			(project ""
 				(path "/96bcf3cc-a3b8-4386-8709-07acaf7b6253/b707efaf-e934-4479-b5a7-a53392b0d81d"
-					(reference "C_INV")
+					(reference "C_INV1")
 					(unit 1)
 				)
@@
 			)
 		)
-		(property "Footprint" ""
+		(property "Footprint" "Capacitor_SMD:C_0402_1005Metric"
 			(at 75.8952 36.83 0)
 			(effects
@@
 			)
 		)
-		(property "Footprint" ""
+		(property "Footprint" "Package_TO_SOT_SMD:SOT-353_SC-70-5"
 			(at 171.45 49.53 0)
 			(effects
@@
 		(dnp no)
 		(fields_autoplaced yes)
-		(property "Reference" "R_DEBOUNCE"
+		(property "Reference" "R_DEBOUNCE1"
 			(at 151.13 133.3499 0)
 			(effects
@@
 			)
 		)
-		(property "Footprint" ""
+		(property "Footprint" "Resistor_SMD:R_0402_1005Metric"
 			(at 146.812 134.62 90)
 			(effects
@@
 			(project ""
 				(path "/96bcf3cc-a3b8-4386-8709-07acaf7b6253/b707efaf-e934-4479-b5a7-a53392b0d81d"
-					(reference "R_DEBOUNCE")
+					(reference "R_DEBOUNCE1")
 					(unit 1)
 				)
@@
 			)
 		)
-		(property "Footprint" ""
+		(property "Footprint" "Resistor_SMD:R_0402_1005Metric"
 			(at 73.152 24.13 90)
 			(effects
@@
 		(dnp no)
 		(fields_autoplaced yes)
-		(property "Reference" "R_ALERT"
+		(property "Reference" "R_ALERT1"
 			(at 208.28 81.2799 0)
 			(effects
@@
 			)
 		)
-		(property "Footprint" ""
+		(property "Footprint" "Resistor_SMD:R_0402_1005Metric"
 			(at 203.962 82.55 90)
 			(effects
@@
 			(project ""
 				(path "/96bcf3cc-a3b8-4386-8709-07acaf7b6253/b707efaf-e934-4479-b5a7-a53392b0d81d"
-					(reference "R_ALERT")
+					(reference "R_ALERT1")
 					(unit 1)
 				)
@@
 			)
 		)
-		(property "Footprint" ""
+		(property "Footprint" "Resistor_SMD:R_0603_1608Metric"
 			(at 112.522 49.53 90)
 			(effects
@@
 		(dnp no)
 		(fields_autoplaced yes)
-		(property "Reference" "C_SCHMITT"
+		(property "Reference" "C_SCHMITT1"
 			(at 176.53 35.5599 0)
 			(effects
@@
 			)
 		)
-		(property "Footprint" ""
+		(property "Footprint" "Capacitor_SMD:C_0402_1005Metric"
 			(at 173.6852 40.64 0)
 			(effects
@@
 			(project ""
 				(path "/96bcf3cc-a3b8-4386-8709-07acaf7b6253/b707efaf-e934-4479-b5a7-a53392b0d81d"
-					(reference "C_SCHMITT")
+					(reference "C_SCHMITT1")
 					(unit 1)
 				)
@@
 			)
 		)
-		(property "Footprint" ""
+		(property "Footprint" "Resistor_SMD:R_0402_1005Metric"
 			(at 217.932 97.79 90)
 			(effects
@@
 			)
 		)
-		(property "Footprint" ""
+		(property "Footprint" "Package_TO_SOT_SMD:SOT-353_SC-70-5"
 			(at 175.26 133.35 0)
 			(effects
@@
 			)
 		)
-		(property "Footprint" "SOT402-1_NXP"
+		(property "Footprint" "Package_SO:TSSOP-14_4.4x5mm_P0.65mm"
 			(at 144.78 87.63 0)
 			(effects
@@
 		(dnp no)
 		(fields_autoplaced yes)
-		(property "Reference" "C_AND"
+		(property "Reference" "C_AND1"
 			(at 191.77 71.1199 0)
 			(effects
@@
 			)
 		)
-		(property "Footprint" ""
+		(property "Footprint" "Capacitor_SMD:C_0402_1005Metric"
 			(at 188.9252 76.2 0)
 			(effects
@@
 			(project ""
 				(path "/96bcf3cc-a3b8-4386-8709-07acaf7b6253/b707efaf-e934-4479-b5a7-a53392b0d81d"
-					(reference "C_AND")
+					(reference "C_AND1")
 					(unit 1)
 				)
@@
 		(dnp no)
 		(fields_autoplaced yes)
-		(property "Reference" "C_DEBOUNCE"
+		(property "Reference" "C_DEBOUNCE1"
 			(at 158.75 140.9699 0)
 			(effects
@@
 			)
 		)
-		(property "Footprint" ""
+		(property "Footprint" "Capacitor_SMD:C_0402_1005Metric"
 			(at 155.9052 146.05 0)
 			(effects
@@
 			(project ""
 				(path "/96bcf3cc-a3b8-4386-8709-07acaf7b6253/b707efaf-e934-4479-b5a7-a53392b0d81d"
-					(reference "C_DEBOUNCE")
-					(unit 1)
-				)
+					(reference "C_DEBOUNCE1")
+					(unit 1)
+				)

Commit message: net labels
Connections:
- net WDT_OUT: now reaches U12.2, U6.3 (OUT)
- net WDT_RST: now reaches R12.2, U6.4 (RESET), U6.8 (VCC)
- net WDT_CONT: now reaches C_CV1.1, U6.5 (CONT)
- net WDT_DISCH: now reaches C15.1, R3.2, U6.6 (THRES), U6.7 (DISCH)
- net WDT_OK: now reaches U12.4, U7.1 (1A)
- net BTN_FILT: now reaches C_DEBOUNCE1.1, R_DEBOUNCE1.2, U13.2
- net AND_1B: now reaches U13.4, U7.2 (1B)
- net AND_3Y: now reaches U7.12 (4A), U7.8 (3Y)
- net AND_1Y: now reaches U7.3 (1Y), U7.4 (2A)
- net LOGIC_2Y: now reaches U7.6 (2Y), U7.9 (3A)
Changed lines of the file:
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@@
+		)
+	)
+	(label "LOGIC_2Y"
+		(at 168.2796 100.33 0)
+		(effects
+			(font
+				(size 1.27 1.27)
+			)
+			(justify left bottom)
+		)
+	)
+	(label "WDT_OUT"
+		(at 161.29 52.1198 0)
+		(effects
+			(font
+				(size 1.27 1.27)
+			)
+			(justify left bottom)
+		)
+	)
+	(label "AND_1Y"
+		(at 144.78 94.1423 0)
+		(effects
+			(font
+				(size 1.27 1.27)
+			)
+			(justify left bottom)
+		)
+	)
+	(label "WDT_CONT"
+		(at 109.22 59.8732 0)
+		(effects
+			(font
+				(size 1.27 1.27)
+			)
+			(justify left bottom)
+		)
+	)
+	(label "BTN_FILT"
+		(at 160.02 136.268 0)
+		(effects
+			(font
+				(size 1.27 1.27)
+			)
+			(justify left bottom)
+		)
+	)
+	(label "WDT_RST"
+		(at 77.039 27.94 0)
+		(effects
+			(font
+				(size 1.27 1.27)
+			)
+			(justify left bottom)
+		)
+	)
+	(label "WDT_DISCH"
+		(at 109.22 53.7566 0)
+		(effects
+			(font
+				(size 1.27 1.27)
+			)
+			(justify left bottom)
+		)
+	)
+	(label "AND_3Y"
+		(at 202.9473 92.71 0)
+		(effects
+			(font
+				(size 1.27 1.27)
+			)
+			(justify left bottom)
+		)
+	)
+	(label "AND_1B"
+		(at 187.96 115.3423 0)
+		(effects
+			(font
+				(size 1.27 1.27)
+			)
+			(justify left bottom)
+		)
+	)
+	(label "WDT_OK"
+		(at 176.5987 49.53 0)
+		(effects
+			(font
+				(size 1.27 1.27)
+			)
+			(justify left bottom)
 		)
 	)
