File: mcu.kicad_sch (KiCad schematic)
At the start: 14 parts, among them U14 AP2112K-3.3, U5 ESP32-S3-WROOM-1-N8R2

Commit message: footprints
Parts:
- C_3V3_1: footprint (none) -> Capacitor_SMD:C_0402_1005Metric
- C_3V3_2: footprint (none) -> Capacitor_SMD:C_0805_2012Metric
- C_LDO_IN1: renamed from C_LDO_IN; footprint (none) -> Capacitor_SMD:C_0805_2012Metric
- C_LDO_OUT1: renamed from C_LDO_OUT; footprint (none) -> Capacitor_SMD:C_0805_2012Metric
- C_RST1: renamed from C_RST; footprint (none) -> Button_Switch_SMD:SW_SPST_TL3342
- R13, R14, R15, R16: footprint (none) -> Resistor_SMD:R_0402_1005Metric
- SW_BOOT1: renamed from SW_BOOT; footprint (none) -> Button_Switch_SMD:SW_SPST_TL3342
- U5: footprint ESP32-S3-WROOM-1_EXP -> RF_Module:ESP32-S3-WROOM-1
- renumbered C_BOOT to C_BOOT_MCU1, SW_RST to SW_RST1
Changed lines of the file:
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@@
 			)
 		)
-		(property "Footprint" ""
+		(property "Footprint" "Resistor_SMD:R_0402_1005Metric"
 			(at 75.692 101.6 90)
 			(effects
@@
 			)
 		)
-		(property "Footprint" ""
+		(property "Footprint" "Capacitor_SMD:C_0402_1005Metric"
 			(at 80.9752 76.2 0)
 			(effects
@@
 			)
 		)
-		(property "Footprint" ""
+		(property "Footprint" "Resistor_SMD:R_0402_1005Metric"
 			(at 75.692 113.03 90)
 			(effects
@@
 			)
 		)
-		(property "Footprint" ""
+		(property "Footprint" "Capacitor_SMD:C_0805_2012Metric"
 			(at 96.2152 76.2 0)
 			(effects
@@
 			)
 		)
-		(property "Footprint" ""
+		(property "Footprint" "Resistor_SMD:R_0402_1005Metric"
 			(at 98.552 95.25 90)
 			(effects
@@
 			)
 		)
-		(property "Footprint" "ESP32-S3-WROOM-1_EXP"
+		(property "Footprint" "RF_Module:ESP32-S3-WROOM-1"
 			(at 113.03 73.66 0)
 			(effects
@@
 		(dnp no)
 		(fields_autoplaced yes)
-		(property "Reference" "C_BOOT"
+		(property "Reference" "C_BOOT_MCU1"
 			(at 177.8 132.0799 0)
 			(effects
@@
 			(project ""
 				(path "/96bcf3cc-a3b8-4386-8709-07acaf7b6253/08b7f495-5348-4df7-a573-a1643fa832c9"
-					(reference "C_BOOT")
+					(reference "C_BOOT_MCU1")
 					(unit 1)
 				)
@@
 		(dnp no)
 		(fields_autoplaced yes)
-		(property "Reference" "C_LDO_IN"
+		(property "Reference" "C_LDO_IN1"
 			(at 49.53 86.3599 0)
 			(effects
@@
 			)
 		)
-		(property "Footprint" ""
+		(property "Footprint" "Capacitor_SMD:C_0805_2012Metric"
 			(at 46.6852 91.44 0)
 			(effects
@@
 			(project ""
 				(path "/96bcf3cc-a3b8-4386-8709-07acaf7b6253/08b7f495-5348-4df7-a573-a1643fa832c9"
-					(reference "C_LDO_IN")
+					(reference "C_LDO_IN1")
 					(unit 1)
 				)
@@
 		(dnp no)
 		(fields_autoplaced yes)
-		(property "Reference" "C_RST"
+		(property "Reference" "C_RST1"
 			(at 86.36 81.2799 0)
 			(effects
@@
 			)
 		)
-		(property "Footprint" ""
+		(property "Footprint" "Button_Switch_SMD:SW_SPST_TL3342"
 			(at 83.5152 86.36 0)
 			(effects
@@
 			(project ""
 				(path "/96bcf3cc-a3b8-4386-8709-07acaf7b6253/08b7f495-5348-4df7-a573-a1643fa832c9"
-					(reference "C_RST")
+					(reference "C_RST1")
 					(unit 1)
 				)
@@
 		(on_board yes)
 		(dnp no)
-		(property "Reference" "SW_BOOT"
+		(property "Reference" "SW_BOOT1"
 			(at 166.37 121.92 0)
 			(effects
@@
 			)
 		)
-		(property "Footprint" ""
+		(property "Footprint" "Button_Switch_SMD:SW_SPST_TL3342"
 			(at 166.37 124.46 0)
 			(effects
@@
 			(project ""
 				(path "/96bcf3cc-a3b8-4386-8709-07acaf7b6253/08b7f495-5348-4df7-a573-a1643fa832c9"
-					(reference "SW_BOOT")
+					(reference "SW_BOOT1")
 					(unit 1)
 				)
@@
 		(dnp no)
 		(fields_autoplaced yes)
-		(property "Reference" "SW_RST"
+		(property "Reference" "SW_RST1"
 			(at 88.9 71.12 0)
 			(effects
@@
 			(project ""
 				(path "/96bcf3cc-a3b8-4386-8709-07acaf7b6253/08b7f495-5348-4df7-a573-a1643fa832c9"
-					(reference "SW_RST")
+					(reference "SW_RST1")
 					(unit 1)
 				)
@@
 		(dnp no)
 		(fields_autoplaced yes)
-		(property "Reference" "C_LDO_OUT"
+		(property "Reference" "C_LDO_OUT1"
 			(at 100.33 86.3599 0)
 			(effects
@@
 			)
 		)
-		(property "Footprint" ""
+		(property "Footprint" "Capacitor_SMD:C_0805_2012Metric"
 			(at 97.4852 91.44 0)
 			(effects
@@
 			(project ""
 				(path "/96bcf3cc-a3b8-4386-8709-07acaf7b6253/08b7f495-5348-4df7-a573-a1643fa832c9"
-					(reference "C_LDO_OUT")
+					(reference "C_LDO_OUT1")
 					(unit 1)
 				)
@@
 			)
 		)
-		(property "Footprint" ""
+		(property "Footprint" "Resistor_SMD:R_0402_1005Metric"
 			(at 104.902 95.25 90)
 			(effects

Commit message: net labels
Connections:
- net ESP_BOOT: now reaches SW_BOOT1.1, U5.27 (IO0)
Changed lines of the file:
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@@
+		)
+	)
+	(label "ESP_BOOT"
+		(at 156.1625 129.54 0)
+		(effects
+			(font
+				(size 1.27 1.27)
+			)
+			(justify left bottom)
 		)
 	)

Commit message: add missing footprints
Parts:
- C_BOOT_MCU1: footprint (none) -> Capacitor_SMD:C_0402_1005Metric
- SW_RST1: footprint (none) -> Button_Switch_SMD:SW_SPST_TL3342
Changed lines of the file:
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@@
 			)
 		)
-		(property "Footprint" ""
+		(property "Footprint" "Capacitor_SMD:C_0402_1005Metric"
 			(at 174.9552 137.16 0)
 			(effects
@@
 			)
 		)
-		(property "Footprint" ""
+		(property "Footprint" "Button_Switch_SMD:SW_SPST_TL3342"
 			(at 88.9 73.66 0)
 			(effects
