File: usb_power.kicad_sch (KiCad schematic)
At the start: 7 parts, among them J2 USB_C_Receptacle_USB2.0_14P

Commit message: footprints
Parts:
- D2: footprint DO-214AASMB_J-BEND_LTF -> Diode_SMD:D_SMB
- D3: footprint DRL5 -> Package_TO_SOT_SMD:SOT-23
- R17, R18: footprint (none) -> Resistor_SMD:R_0402_1005Metric
Changed lines of the file:
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@@
 			)
 		)
-		(property "Footprint" ""
+		(property "Footprint" "Resistor_SMD:R_0402_1005Metric"
 			(at 74.422 92.71 90)
 			(effects
@@
 			)
 		)
-		(property "Footprint" "DRL5"
+		(property "Footprint" "Package_TO_SOT_SMD:SOT-23"
 			(at 78.74 102.87 0)
 			(effects
@@
 			)
 		)
-		(property "Footprint" "DO-214AASMB_J-BEND_LTF"
+		(property "Footprint" "Diode_SMD:D_SMB"
 			(at 92.71 91.44 0)
 			(effects
@@
 			)
 		)
-		(property "Footprint" ""
+		(property "Footprint" "Resistor_SMD:R_0402_1005Metric"
 			(at 82.042 91.44 90)
 			(effects

Commit message: net labels
Connections:
- net USB_CC2: now reaches J2.B5 (CC2), R18.1
- net USB_CC1: now reaches J2.A5 (CC1), R17.1
Changed lines of the file:
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@@
+		)
+	)
+	(label "USB_CC2"
+		(at 73.4802 92.71 0)
+		(effects
+			(font
+				(size 1.27 1.27)
+			)
+			(justify left bottom)
+		)
+	)
+	(label "USB_CC1"
+		(at 74.0127 87.63 0)
+		(effects
+			(font
+				(size 1.27 1.27)
+			)
+			(justify left bottom)
 		)
 	)

Commit message: yay
Parts:
- D3: footprint Package_TO_SOT_SMD:SOT-23 -> Package_TO_SOT_SMD:SOT-23-5
Changed lines of the file:
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@@
 			)
 		)
-		(property "Footprint" "Package_TO_SOT_SMD:SOT-23"
+		(property "Footprint" "Package_TO_SOT_SMD:SOT-23-5"
 			(at 78.74 102.87 0)
 			(effects
